File: deska.brd (EAGLE design)
At the start: 50.5 x 47 mm, 6 parts

Commit message: uprava desky
Parts:
- added SL2: (no value), con-amp-quick:02P
- moved SI7021 15.3 mm to (41.9, 7.62)
- moved U$1 1.27 mm to (33.0, 35.6)
Connections:
- net N$1 renamed RESET
- net N$2 renamed CE
- net N$3 renamed DC
- net N$4 renamed DIN
- net N$5 renamed CLK
- removed net N$6: SI7021.3, U$1.A6
- removed net N$7: SI7021.4, U$1.A5
- new net SCL: SI7021.3, SL2.1, U$1.A5
- new net SDA: SI7021.4, SL2.2, U$1.A4
- net +5V: now also U$1.GND1
- net GND: now also U$1.GND
Routing:
- net +5V: track 66.0 -> 111.1 mm
- net GND: track 99.7 -> 137.8 mm
- net SCL: track 0.00 -> 34.3 mm
- net SDA: track 0.00 -> 29.2 mm
- net N$6: track 21.6 -> 0.00 mm
- net N$7: track 16.5 -> 0.00 mm
- net RESET: track 20.3 -> 21.6 mm
- net CE: track 20.3 -> 21.6 mm
- net DIN: track 45.7 -> 47.0 mm
- net DC: track 20.3 -> 21.6 mm
- net CLK: track 35.6 -> 36.8 mm
Other:
- board size 50.5 x 47 mm -> 50.5 x 49.5 mm

Commit message: +deska +ino
Parts:
- moved R1 15.9 mm to (35.6, 20.3)
- moved SL1 9.25 mm to (26.7, 15.2)
- moved DS18B20 6.35 mm to (17.8, 6.35)
- moved SI7021 2.84 mm to (43.2, 5.08), turned to 90 degrees
- moved U$1 2.84 mm to (34.3, 33.0)
- moved X1 2.54 mm to (5.08, 6.35)
- moved SL2 1.80 mm to (40.6, 31.8), turned to 270 degrees
Connections:
- net +5V: now also U$1.VCC; no longer U$1.GND1
- net GND: now also DS18B20.2; no longer DS18B20.1
- net N$8: now also DS18B20.1, U$1.D9; no longer DS18B20.2
Routing:
- net N$8: track 8.26 -> 38.6 mm
- net +5V: track 111.1 -> 132.7 mm
- net GND: track 137.8 -> 155.4 mm
- net CLK: track 36.8 -> 27.7 mm
- net RESET: track 21.6 -> 12.5 mm
- net CE: track 21.6 -> 12.5 mm
- net DC: track 21.6 -> 12.5 mm
- net DIN: track 47.0 -> 38.6 mm
- net SCL: track 34.3 -> 39.4 mm
Other:
- board size 50.5 x 49.5 mm -> 49.2 x 47 mm
