File: deska.sch (EAGLE design)
At the start: 6 parts

Commit message: uprava desky
Parts:
- added SL2: (no value), con-amp-quick:M02
Connections:
- net N$1 renamed RESET
- net N$2 renamed CE
- net N$3 renamed DC
- net N$4 renamed DIN
- net N$5 renamed CLK
- removed net N$6: SI7021.3, U$1.A6
- removed net N$7: SI7021.4, U$1.A5
- new net SCL: SI7021.3, SL2.1, U$1.A5
- new net SDA: SI7021.4, SL2.2, U$1.A4
- net +5V: now also U$1.GND2
- net GND: now also U$1.GND
Changed lines of the file:
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@@
 <part name="GND4" library="supply1" deviceset="GND" device=""/>
 <part name="R1" library="rcl" deviceset="R-EU_" device="0207/10" value="4K7"/>
+<part name="SL2" library="con-amp-quick" deviceset="M02" device=""/>
+<part name="P+5" library="supply1" deviceset="+5V" device=""/>
+<part name="GND5" library="supply1" deviceset="GND" device=""/>
 </parts>
 <sheets>
@@
 <instance part="GND4" gate="1" x="116.84" y="25.4"/>
 <instance part="R1" gate="G$1" x="106.68" y="55.88" rot="R90"/>
+<instance part="SL2" gate="G$1" x="106.68" y="33.02" rot="R180"/>
+<instance part="P+5" gate="1" x="10.16" y="48.26" rot="R90"/>
+<instance part="GND5" gate="1" x="58.42" y="50.8"/>
 </instances>
 <busses>
 </busses>
 <nets>
-<net name="N$1" class="0">
+<net name="RESET" class="0">
 <segment>
 <pinref part="U$1" gate="G$1" pin="D3"/>
@@
 </segment>
 </net>
-<net name="N$2" class="0">
+<net name="CE" class="0">
 <segment>
 <pinref part="U$1" gate="G$1" pin="D4"/>
@@
 </segment>
 </net>
-<net name="N$3" class="0">
+<net name="DC" class="0">
 <segment>
 <pinref part="U$1" gate="G$1" pin="D5"/>
@@
 </segment>
 </net>
-<net name="N$4" class="0">
+<net name="DIN" class="0">
 <segment>
 <pinref part="U$1" gate="G$1" pin="D11"/>
@@
 </segment>
 </net>
-<net name="N$5" class="0">
+<net name="CLK" class="0">
 <segment>
 <pinref part="U$1" gate="G$1" pin="D13"/>
@@
 <pinref part="GND4" gate="1" pin="GND"/>
 </segment>
+<segment>
+<pinref part="U$1" gate="G$1" pin="GND"/>
+<pinref part="GND5" gate="1" pin="GND"/>
+<wire x1="53.34" y1="53.34" x2="58.42" y2="53.34" width="0.1524" layer="91"/>
+</segment>
 </net>
 <net name="+5V" class="0">
@@
 <pinref part="P+4" gate="1" pin="+5V"/>
 </segment>
+<segment>
+<pinref part="U$1" gate="G$1" pin="GND2"/>
+<pinref part="P+5" gate="1" pin="+5V"/>
+</segment>
 </net>
-<net name="N$6" class="0">
+<net name="SCL" class="0">
 <segment>
 <pinref part="SI7021" gate="G$1" pin="3"/>
-<wire x1="35.56" y1="12.7" x2="93.98" y2="12.7" width="0.1524" layer="91"/>
-<wire x1="93.98" y1="12.7" x2="93.98" y2="73.66" width="0.1524" layer="91"/>
-<pinref part="U$1" gate="G$1" pin="A6"/>
-<wire x1="35.56" y1="17.78" x2="35.56" y2="12.7" width="0.1524" layer="91"/>
+<wire x1="33.02" y1="12.7" x2="93.98" y2="12.7" width="0.1524" layer="91"/>
+<wire x1="93.98" y1="12.7" x2="93.98" y2="33.02" width="0.1524" layer="91"/>
+<pinref part="U$1" gate="G$1" pin="A5"/>
+<wire x1="93.98" y1="33.02" x2="93.98" y2="73.66" width="0.1524" layer="91"/>
+<wire x1="33.02" y1="12.7" x2="33.02" y2="17.78" width="0.1524" layer="91"/>
+<pinref part="SL2" gate="G$1" pin="1"/>
+<wire x1="99.06" y1="33.02" x2="93.98" y2="33.02" width="0.1524" layer="91"/>
+<junction x="93.98" y="33.02"/>
 </segment>
 </net>
-<net name="N$7" class="0">
+<net name="SDA" class="0">
 <segment>
 <pinref part="SI7021" gate="G$1" pin="4"/>
-<wire x1="33.02" y1="15.24" x2="96.52" y2="15.24" width="0.1524" layer="91"/>
-<wire x1="96.52" y1="15.24" x2="96.52" y2="73.66" width="0.1524" layer="91"/>
-<pinref part="U$1" gate="G$1" pin="A5"/>
-<wire x1="33.02" y1="15.24" x2="33.02" y2="17.78" width="0.1524" layer="91"/>
+<wire x1="30.48" y1="15.24" x2="96.52" y2="15.24" width="0.1524" layer="91"/>
+<wire x1="96.52" y1="15.24" x2="96.52" y2="30.48" width="0.1524" layer="91"/>
+<pinref part="U$1" gate="G$1" pin="A4"/>
+<wire x1="96.52" y1="30.48" x2="96.52" y2="73.66" width="0.1524" layer="91"/>
+<wire x1="30.48" y1="17.78" x2="30.48" y2="15.24" width="0.1524" layer="91"/>
+<pinref part="SL2" gate="G$1" pin="2"/>
+<wire x1="99.06" y1="30.48" x2="96.52" y2="30.48" width="0.1524" layer="91"/>
+<junction x="96.52" y="30.48"/>
 </segment>
 </net>

Commit message: +deska +ino
Connections:
- net +5V: now also U$1.VCC; no longer U$1.GND2
- net GND: now also DS18B20-2.KL; no longer DS18B20-1.KL
- net N$8: now also DS18B20-1.KL, U$1.D9; no longer DS18B20-2.KL
Changed lines of the file:
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@@
 <?xml version="1.0" encoding="utf-8"?>
 <!DOCTYPE eagle SYSTEM "eagle.dtd">
-<eagle version="7.7.0">
+<eagle version="7.3.0">
 <drawing>
 <settings>
@@
 <instance part="DS18B20" gate="-3" x="121.92" y="60.96" rot="R180"/>
 <instance part="P+2" gate="1" x="99.06" y="60.96" rot="R90"/>
-<instance part="GND2" gate="1" x="114.3" y="45.72"/>
+<instance part="GND2" gate="1" x="114.3" y="53.34"/>
 <instance part="SI7021" gate="G$1" x="91.44" y="78.74" rot="R270"/>
 <instance part="P+3" gate="1" x="88.9" y="71.12" rot="R180"/>
@@
 <instance part="R1" gate="G$1" x="106.68" y="55.88" rot="R90"/>
 <instance part="SL2" gate="G$1" x="106.68" y="33.02" rot="R180"/>
-<instance part="P+5" gate="1" x="10.16" y="48.26" rot="R90"/>
+<instance part="P+5" gate="1" x="58.42" y="40.64" rot="R180"/>
 <instance part="GND5" gate="1" x="58.42" y="50.8"/>
 </instances>
@@
 </segment>
 <segment>
-<pinref part="GND2" gate="1" pin="GND"/>
-<wire x1="114.3" y1="48.26" x2="114.3" y2="50.8" width="0.1524" layer="91"/>
-<pinref part="DS18B20" gate="-1" pin="KL"/>
-<wire x1="114.3" y1="50.8" x2="116.84" y2="50.8" width="0.1524" layer="91"/>
-</segment>
-<segment>
 <pinref part="SI7021" gate="G$1" pin="2"/>
 <pinref part="GND3" gate="1" pin="GND"/>
@@
 <pinref part="GND5" gate="1" pin="GND"/>
 <wire x1="53.34" y1="53.34" x2="58.42" y2="53.34" width="0.1524" layer="91"/>
+</segment>
+<segment>
+<pinref part="DS18B20" gate="-2" pin="KL"/>
+<pinref part="GND2" gate="1" pin="GND"/>
+<wire x1="116.84" y1="55.88" x2="114.3" y2="55.88" width="0.1524" layer="91"/>
 </segment>
 </net>
@@
 </segment>
 <segment>
-<pinref part="U$1" gate="G$1" pin="GND2"/>
+<pinref part="U$1" gate="G$1" pin="VCC"/>
 <pinref part="P+5" gate="1" pin="+5V"/>
+<wire x1="53.34" y1="48.26" x2="58.42" y2="48.26" width="0.1524" layer="91"/>
+<wire x1="58.42" y1="48.26" x2="58.42" y2="43.18" width="0.1524" layer="91"/>
 </segment>
 </net>
@@
 <segment>
 <pinref part="R1" gate="G$1" pin="1"/>
-<wire x1="106.68" y1="50.8" x2="111.76" y2="50.8" width="0.1524" layer="91"/>
-<wire x1="111.76" y1="50.8" x2="111.76" y2="55.88" width="0.1524" layer="91"/>
-<pinref part="DS18B20" gate="-2" pin="KL"/>
-<wire x1="111.76" y1="55.88" x2="116.84" y2="55.88" width="0.1524" layer="91"/>
-</segment>
-</net>
+<pinref part="DS18B20" gate="-1" pin="KL"/>
+<wire x1="106.68" y1="50.8" x2="116.84" y2="50.8" width="0.1524" layer="91"/>
+<wire x1="91.44" y1="10.16" x2="91.44" y2="50.8" width="0.1524" layer="91"/>
+<wire x1="91.44" y1="50.8" x2="106.68" y2="50.8" width="0.1524" layer="91"/>
+<junction x="106.68" y="50.8"/>
+<pinref part="U$1" gate="G$1" pin="D9"/>
+<wire x1="12.7" y1="27.94" x2="12.7" y2="10.16" width="0.1524" layer="91"/>
+<wire x1="12.7" y1="10.16" x2="91.44" y2="10.16" width="0.1524" layer="91"/>
+</segment>
+</net>
